File: cad/power.sch (KiCad schematic (older format))
At the start: 30 parts

Commit message: passed erc
Parts:
- gave numbers to parts that had none: 30
Connections:
- wire segments 48 -> 52
Changed lines of the file:
@@
 $EndDescr
 $Comp
-L C C?
+L C C20
 U 1 1 548DFC7F
 P 3950 2600
-F 0 "C?" H 4000 2700 50  0000 L CNN
+F 0 "C20" H 4000 2700 50  0000 L CNN
 F 1 "1uF" H 4000 2500 50  0000 L CNN
 F 2 "" H 3950 2600 60  0000 C CNN
@@
 $EndComp
 $Comp
-L BATTERY BT?
+L BATTERY BT1
 U 1 1 548DFD04
 P 6850 6150
-F 0 "BT?" H 6850 6350 50  0000 C CNN
+F 0 "BT1" H 6850 6350 50  0000 C CNN
 F 1 "BATTERY" H 6850 5960 50  0000 C CNN
 F 2 "" H 6850 6150 60  0000 C CNN
@@
 Connection ~ 3950 2400
 $Comp
-L C C?
+L C C22
 U 1 1 548E039E
 P 4700 3300
-F 0 "C?" H 4750 3400 50  0000 L CNN
+F 0 "C22" H 4750 3400 50  0000 L CNN
 F 1 "10nF" H 4750 3200 50  0000 L CNN
 F 2 "" H 4700 3300 60  0000 C CNN
@@
 $EndComp
 $Comp
-L C C?
+L C C26
 U 1 1 548E0BCE
 P 7000 2600
-F 0 "C?" H 7050 2700 50  0000 L CNN
+F 0 "C26" H 7050 2700 50  0000 L CNN
 F 1 "4.7uF" H 7050 2500 50  0000 L CNN
 F 2 "" H 7000 2600 60  0000 C CNN
@@
 $EndComp
 $Comp
-L TPS37001 U?
+L TPS37001 U3
 U 1 1 548E19BC
 P 5250 2500
-F 0 "U?" H 5200 2750 60  0000 C CNN
+F 0 "U3" H 5200 2750 60  0000 C CNN
 F 1 "TPS37001" H 5500 2250 60  0000 C CNN
 F 2 "" H 5250 2500 60  0000 C CNN
@@
 $EndComp
 $Comp
-L R R?
+L R R14
 U 1 1 548E3182
 P 5550 3200
-F 0 "R?" V 5630 3200 50  0000 C CNN
+F 0 "R14" V 5630 3200 50  0000 C CNN
 F 1 "0" V 5550 3200 50  0000 C CNN
 F 2 "" H 5550 3200 60  0000 C CNN
@@
 	5200 3200 5200 3300
 $Comp
-L R R?
+L R R16
 U 1 1 548E3B5C
 P 6200 2650
-F 0 "R?" V 6280 2650 50  0000 C CNN
+F 0 "R16" V 6280 2650 50  0000 C CNN
 F 1 "39k" V 6200 2650 50  0000 C CNN
 F 2 "" H 6200 2650 60  0000 C CNN
@@
 $EndComp
 $Comp
-L R R?
+L R R17
 U 1 1 548E3BAD
 P 6200 3250
-F 0 "R?" V 6280 3250 50  0000 C CNN
+F 0 "R17" V 6280 3250 50  0000 C CNN
 F 1 "30k" V 6200 3250 50  0000 C CNN
 F 2 "" H 6200 3250 60  0000 C CNN
@@
 $EndComp
 $Comp
-L C C?
+L C C24
 U 1 1 548E476C
 P 6500 2650
-F 0 "C?" H 6550 2750 50  0000 L CNN
+F 0 "C24" H 6550 2750 50  0000 L CNN
 F 1 "22pF" H 6550 2550 50  0000 L CNN
 F 2 "" H 6500 2650 60  0000 C CNN
@@
 EN
 $Comp
-L C C?
+L C C21
 U 1 1 548E9E6E
 P 3950 4000
-F 0 "C?" H 4000 4100 50  0000 L CNN
+F 0 "C21" H 4000 4100 50  0000 L CNN
 F 1 "4.7uF" H 4000 3900 50  0000 L CNN
 F 2 "" H 3950 4000 60  0000 C CNN
@@
 $EndComp
 $Comp
-L C C?
+L C C23
 U 1 1 548E9E82
 P 4700 4700
-F 0 "C?" H 4750 4800 50  0000 L CNN
+F 0 "C23" H 4750 4800 50  0000 L CNN
 F 1 "10nF" H 4750 4600 50  0000 L CNN
 F 2 "" H 4700 4700 60  0000 C CNN
@@
 $EndComp
 $Comp
-L C C?
+L C C27
 U 1 1 548E9E8E
 P 7000 4000
-F 0 "C?" H 7050 4100 50  0000 L CNN
+F 0 "C27" H 7050 4100 50  0000 L CNN
 F 1 "4.7uF" H 7050 3900 50  0000 L CNN
 F 2 "" H 7000 4000 60  0000 C CNN
@@
 $EndComp
 $Comp
-L TPS37001 U?
+L TPS37001 U4
 U 1 1 548E9E9A
 P 5250 3900
-F 0 "U?" H 5200 4150 60  0000 C CNN
+F 0 "U4" H 5200 4150 60  0000 C CNN
 F 1 "TPS37001" H 5500 3650 60  0000 C CNN
 F 2 "" H 5250 3900 60  0000 C CNN
@@
 $EndComp
 $Comp
-L R R?
+L R R15
 U 1 1 548E9EB5
 P 5550 4600
-F 0 "R?" V 5630 4600 50  0000 C CNN
+F 0 "R15" V 5630 4600 50  0000 C CNN
 F 1 "0" V 5550 4600 50  0000 C CNN
 F 2 "" H 5550 4600 60  0000 C CNN
@@
 	5200 4600 5200 4700
 $Comp
-L R R?
+L R R18
 U 1 1 548E9EBF
 P 6200 4050
-F 0 "R?" V 6280 4050 50  0000 C CNN
+F 0 "R18" V 6280 4050 50  0000 C CNN
 F 1 "39k" V 6200 4050 50  0000 C CNN
 F 2 "" H 6200 4050 60  0000 C CNN
@@
 $EndComp
 $Comp
-L R R?
+L R R19
 U 1 1 548E9EC5
 P 6200 4650
-F 0 "R?" V 6280 4650 50  0000 C CNN
+F 0 "R19" V 6280 4650 50  0000 C CNN
 F 1 "30k" V 6200 4650 50  0000 C CNN
 F 2 "" H 6200 4650 60  0000 C CNN
@@
 $EndComp
 $Comp
-L C C?
+L C C25
 U 1 1 548E9ECB
 P 6500 4050
-F 0 "C?" H 6550 4150 50  0000 L CNN
+F 0 "C25" H 6550 4150 50  0000 L CNN
 F 1 "22pF" H 6550 3950 50  0000 L CNN
 F 2 "" H 6500 4050 60  0000 C CNN
@@
 $EndComp
 $Comp
-L R R?
+L R R11
 U 1 1 548F0D05
 P 3550 3800
-F 0 "R?" V 3630 3800 50  0000 C CNN
+F 0 "R11" V 3630 3800 50  0000 C CNN
 F 1 "10" V 3550 3800 50  0000 C CNN
 F 2 "" H 3550 3800 60  0000 C CNN
@@
 $EndComp
 $Comp
-L C C?
+L C C17
 U 1 1 548F108E
 P 2800 4000
-F 0 "C?" H 2850 4100 50  0000 L CNN
+F 0 "C17" H 2850 4100 50  0000 L CNN
 F 1 "4.7uF" H 2850 3900 50  0000 L CNN
 F 2 "" H 2800 4000 60  0000 C CNN
@@
 $EndComp
 $Comp
-L C C?
+L C C18
 U 1 1 548F10FD
 P 3150 4000
-F 0 "C?" H 3200 4100 50  0000 L CNN
+F 0 "C18" H 3200 4100 50  0000 L CNN
 F 1 "100nF" H 3200 3900 50  0000 L CNN
 F 2 "" H 3150 4000 60  0000 C CNN
@@
 $EndComp
 $Comp
-L SW_PUSH SW?
+L SW_PUSH SW1
 U 1 1 548F8D37
 P 1750 6250
-F 0 "SW?" H 1900 6360 50  0000 C CNN
+F 0 "SW1" H 1900 6360 50  0000 C CNN
 F 1 "SW_PUSH" H 1750 6170 50  0000 C CNN
 F 2 "" H 1750 6250 60  0000 C CNN
@@
 EN
 $Comp
-L DIODE D?
+L DIODE D3
 U 1 1 548FA9F5
 P 2450 5700
-F 0 "D?" H 2450 5800 40  0000 C CNN
+F 0 "D3" H 2450 5800 40  0000 C CNN
 F 1 "DIODE" H 2450 5600 40  0000 C CNN
 F 2 "" H 2450 5700 60  0000 C CNN
@@
 Connection ~ 2650 6250
 $Comp
-L R R?
+L R R10
 U 1 1 548FBD41
 P 2850 6500
-F 0 "R?" V 2930 6500 50  0000 C CNN
+F 0 "R10" V 2930 6500 50  0000 C CNN
 F 1 "100k" V 2850 6500 50  0000 C CNN
 F 2 "" H 2850 6500 60  0000 C CNN
@@
 BUTTON
 $Comp
-L ZENER D?
+L ZENER D2
 U 1 1 548FCC83
 P 2150 7050
-F 0 "D?" H 2150 7150 50  0000 C CNN
+F 0 "D2" H 2150 7150 50  0000 C CNN
 F 1 "ZENER" H 2150 6950 40  0000 C CNN
 F 2 "" H 2150 7050 60  0000 C CNN
@@
 $EndComp
 $Comp
-L R R?
+L R R8
 U 1 1 548FCD4A
 P 2150 6500
-F 0 "R?" V 2230 6500 50  0000 C CNN
+F 0 "R8" V 2230 6500 50  0000 C CNN
 F 1 "2k2" V 2150 6500 50  0000 C CNN
 F 2 "" H 2150 6500 60  0000 C CNN
@@
 Connection ~ 2150 6800
 $Comp
-L C C?
+L C C19
 U 1 1 54900A66
 P 3150 6450
-F 0 "C?" H 3200 6550 50  0000 L CNN
+F 0 "C19" H 3200 6550 50  0000 L CNN
 F 1 "10nF" H 3200 6350 50  0000 L CNN
 F 2 "" H 3150 6450 60  0000 C CNN
@@
 $EndComp
 $Comp
-L DIODE D?
+L DIODE D4
 U 1 1 54900D4C
 P 2450 6250
-F 0 "D?" H 2450 6350 40  0000 C CNN
+F 0 "D4" H 2450 6350 40  0000 C CNN
 F 1 "DIODE" H 2450 6150 40  0000 C CNN
 F 2 "" H 2450 6250 60  0000 C CNN
@@
 Connection ~ 3150 6250
 $Comp
-L R R?
+L R R9
 U 1 1 5490905D
 P 2450 7050
-F 0 "R?" V 2530 7050 50  0000 C CNN
+F 0 "R9" V 2530 7050 50  0000 C CNN
 F 1 "20k" V 2450 7050 50  0000 C CNN
 F 2 "" H 2450 7050 60  0000 C CNN
@@
 $EndComp
 $Comp
-L R R?
+L R R13
 U 1 1 5490C83D
 P 5300 6850
-F 0 "R?" V 5380 6850 50  0000 C CNN
+F 0 "R13" V 5380 6850 50  0000 C CNN
 F 1 "62k" V 5300 6850 50  0000 C CNN
 F 2 "" H 5300 6850 60  0000 C CNN
@@
 $EndComp
 $Comp
-L R R?
+L R R12
 U 1 1 5490C8BE
 P 5300 6250
-F 0 "R?" V 5380 6250 50  0000 C CNN
+F 0 "R12" V 5380 6250 50  0000 C CNN
 F 1 "36k" V 5300 6250 50  0000 C CNN
 F 2 "" H 5300 6250 60  0000 C CNN
@@
 	4900 6550 5300 6550
 Connection ~ 5300 6550
+$Comp
+L DGND #PWR061
+U 1 1 549476C0
+P 9100 6250
+F 0 "#PWR061" H 9100 6250 40  0001 C CNN
+F 1 "DGND" H 9100 6180 40  0000 C CNN
+F 2 "" H 9100 6250 60  0000 C CNN
+F 3 "" H 9100 6250 60  0000 C CNN
+	1    9100 6250
+	1    0    0    -1
+$EndComp
+$Comp
+L AGND #PWR062
+U 1 1 5494776A
+P 8800 6250
+F 0 "#PWR062" H 8800 6250 40  0001 C CNN
+F 1 "AGND" H 8800 6180 50  0000 C CNN
+F 2 "" H 8800 6250 60  0000 C CNN
+F 3 "" H 8800 6250 60  0000 C CNN
+	1    8800 6250
+	1    0    0    -1
+$EndComp
+$Comp
+L GND #PWR063
+U 1 1 54947D00
+P 8450 6250
+F 0 "#PWR063" H 8450 6250 30  0001 C CNN
+F 1 "GND" H 8450 6180 30  0001 C CNN
+F 2 "" H 8450 6250 60  0000 C CNN
+F 3 "" H 8450 6250 60  0000 C CNN
+	1    8450 6250
+	1    0    0    -1
+$EndComp
+$Comp
+L +BATT #PWR064
+U 1 1 54947D5A
+P 9650 6050
+F 0 "#PWR064" H 9650 6000 20  0001 C CNN
+F 1 "+BATT" H 9650 6150 30  0000 C CNN
+F 2 "" H 9650 6050 60  0000 C CNN
+F 3 "" H 9650 6050 60  0000 C CNN
+	1    9650 6050
+	1    0    0    -1
+$EndComp
+$Comp
+L PWR_FLAG #FLG065
+U 1 1 54947D8C
+P 8450 6150
+F 0 "#FLG065" H 8450 6245 30  0001 C CNN
+F 1 "PWR_FLAG" H 8450 6330 30  0000 C CNN
+F 2 "" H 8450 6150 60  0000 C CNN
+F 3 "" H 8450 6150 60  0000 C CNN
+	1    8450 6150
+	1    0    0    -1
+$EndComp
+$Comp
+L PWR_FLAG #FLG066
+U 1 1 54947DBE
+P 8800 6150
+F 0 "#FLG066" H 8800 6245 30  0001 C CNN
+F 1 "PWR_FLAG" H 8800 6330 30  0000 C CNN
+F 2 "" H 8800 6150 60  0000 C CNN
+F 3 "" H 8800 6150 60  0000 C CNN
+	1    8800 6150
+	1    0    0    -1
+$EndComp
+$Comp
+L PWR_FLAG #FLG067
+U 1 1 54947DF0
+P 9100 6150
+F 0 "#FLG067" H 9100 6245 30  0001 C CNN
+F 1 "PWR_FLAG" H 9100 6330 30  0000 C CNN
+F 2 "" H 9100 6150 60  0000 C CNN
+F 3 "" H 9100 6150 60  0000 C CNN
+	1    9100 6150
+	1    0    0    -1
+$EndComp
+$Comp
+L PWR_FLAG #FLG068
+U 1 1 54947E22
+P 9650 6200
+F 0 "#FLG068" H 9650 6295 30  0001 C CNN
+F 1 "PWR_FLAG" H 9650 6380 30  0000 C CNN
+F 2 "" H 9650 6200 60  0000 C CNN
+F 3 "" H 9650 6200 60  0000 C CNN
+	1    9650 6200
+	-1   0    0    1
+$EndComp
+Wire Wire Line
+	9650 6050 9650 6200
+Wire Wire Line
+	9100 6150 9100 6250
+Wire Wire Line
+	8800 6250 8800 6150
+Wire Wire Line
+	8450 6150 8450 6250
+$Comp
+L PWR_FLAG #FLG069
+U 1 1 5494A391
+P 4200 3800
+F 0 "#FLG069" H 4200 3895 30  0001 C CNN
+F 1 "PWR_FLAG" H 4200 3980 30  0000 C CNN
+F 2 "" H 4200 3800 60  0000 C CNN
+F 3 "" H 4200 3800 60  0000 C CNN
+	1    4200 3800
+	1    0    0    -1
+$EndComp
+Connection ~ 4200 3800
 $EndSCHEMATC

Commit message: did stuff here, not exactly sure what
Parts:
- removed D3, D4: DIODE, symbol DIODE
- added D3: BAT54C, symbol BAT54C
Connections:
- wire segments 52 -> 54
Other:
- moved on the sheet: C17, C18, C21, C23, C25, C27, R11, R15, R18, R19

Commit message: selecting parts for the little passives
Parts:
- removed U3, U4: TPS37001, symbol TPS37001
- added U3, U4: TPS73001, symbol TPS73001
- C24: MPN (none) -> CL05C220JB5NNNC
- C26: MPN (none) -> CL10B475KQ8NQNC
- D2: value ZENER -> 2.7v; MPN (none) -> MM3Z2V7T1G
- R10: MPN (none) -> MCR01MRTF1003
- R11: MPN (none) -> MCR01MRTF10R0
- R12: MPN (none) -> MCR01MRTF3602
- R13: MPN (none) -> MCR01MRTJ623
- R14: MPN (none) -> RC1005J000CS
- R16: MPN (none) -> RC1005J393CS
- R17: MPN (none) -> RC1005J303CS
- R8: MPN (none) -> RMCF0402JT2K20
- R9: MPN (none) -> MCR01MRTF2002
Changed lines of the file:
@@
 F 2 "" H 7000 2600 60  0000 C CNN
 F 3 "" H 7000 2600 60  0000 C CNN
+F 4 "CL10B475KQ8NQNC" H 7000 2600 60  0001 C CNN "MPN"
 	1    7000 2600
 	1    0    0    -1
@@
 	1    0    0    -1
 $EndComp
-$Comp
-L TPS37001 U3
-U 1 1 548E19BC
-P 5250 2500
-F 0 "U3" H 5200 2750 60  0000 C CNN
-F 1 "TPS37001" H 5500 2250 60  0000 C CNN
-F 2 "" H 5250 2500 60  0000 C CNN
-F 3 "" H 5250 2500 60  0000 C CNN
-	1    5250 2500
-	1    0    0    -1
-$EndComp
 Wire Wire Line
 	3950 2400 4750 2400
@@
 F 2 "" H 5550 3200 60  0000 C CNN
 F 3 "" H 5550 3200 60  0000 C CNN
+F 4 "RC1005J000CS" V 5550 3200 60  0001 C CNN "MPN"
 	1    5550 3200
 	0    1    1    0
@@
 F 2 "" H 6200 2650 60  0000 C CNN
 F 3 "" H 6200 2650 60  0000 C CNN
+F 4 "RC1005J393CS" V 6200 2650 60  0001 C CNN "MPN"
 	1    6200 2650
 	1    0    0    -1
@@
 F 2 "" H 6200 3250 60  0000 C CNN
 F 3 "" H 6200 3250 60  0000 C CNN
+F 4 "RC1005J303CS" V 6200 3250 60  0001 C CNN "MPN"
 	1    6200 3250
 	1    0    0    -1
@@
 F 2 "" H 6500 2650 60  0000 C CNN
 F 3 "" H 6500 2650 60  0000 C CNN
+F 4 "CL05C220JB5NNNC" H 6500 2650 60  0001 C CNN "MPN"
 	1    6500 2650
 	1    0    0    -1
@@
 F 3 "" H 7000 4150 60  0000 C CNN
 	1    7000 4150
-	1    0    0    -1
-$EndComp
-$Comp
-L TPS37001 U4
-U 1 1 548E9E9A
-P 5250 4050
-F 0 "U4" H 5200 4300 60  0000 C CNN
-F 1 "TPS37001" H 5500 3800 60  0000 C CNN
-F 2 "" H 5250 4050 60  0000 C CNN
-F 3 "" H 5250 4050 60  0000 C CNN
-	1    5250 4050
 	1    0    0    -1
 $EndComp
@@
 F 2 "" H 3550 3950 60  0000 C CNN
 F 3 "" H 3550 3950 60  0000 C CNN
+F 4 "MCR01MRTF10R0" V 3550 3950 60  0001 C CNN "MPN"
 	1    3550 3950
 	0    1    1    0
@@
 F 2 "" H 2850 6500 60  0000 C CNN
 F 3 "" H 2850 6500 60  0000 C CNN
+F 4 "MCR01MRTF1003" V 2850 6500 60  0001 C CNN "MPN"
 	1    2850 6500
 	1    0    0    -1
@@
 P 2150 7050
 F 0 "D2" H 2150 7150 50  0000 C CNN
-F 1 "ZENER" H 2150 6950 40  0000 C CNN
+F 1 "2.7v" H 2150 6950 40  0000 C CNN
 F 2 "" H 2150 7050 60  0000 C CNN
 F 3 "" H 2150 7050 60  0000 C CNN
+F 4 "MM3Z2V7T1G" H 2150 7050 60  0001 C CNN "MPN"
 	1    2150 7050
 	0    -1   -1   0
@@
 F 2 "" H 2150 6500 60  0000 C CNN
 F 3 "" H 2150 6500 60  0000 C CNN
+F 4 "RMCF0402JT2K20" V 2150 6500 60  0001 C CNN "MPN"
 	1    2150 6500
 	1    0    0    -1
@@
 F 2 "" H 2450 7050 60  0000 C CNN
 F 3 "" H 2450 7050 60  0000 C CNN
+F 4 "MCR01MRTF2002" V 2450 7050 60  0001 C CNN "MPN"
 	1    2450 7050
 	1    0    0    -1
@@
 F 2 "" H 5300 6850 60  0000 C CNN
 F 3 "" H 5300 6850 60  0000 C CNN
+F 4 "MCR01MRTJ623" V 5300 6850 60  0001 C CNN "MPN"
 	1    5300 6850
 	1    0    0    -1
@@
 F 2 "" H 5300 6250 60  0000 C CNN
 F 3 "" H 5300 6250 60  0000 C CNN
+F 4 "MCR01MRTF3602" V 5300 6250 60  0001 C CNN "MPN"
 	1    5300 6250
 	1    0    0    -1
@@
 Wire Wire Line
 	3150 6150 3150 6250
+$Comp
+L TPS73001 U3
+U 1 1 54944F99
+P 5250 2500
+F 0 "U3" H 5200 2750 60  0000 C CNN
+F 1 "TPS73001" H 5500 2250 60  0000 C CNN
+F 2 "" H 5250 2500 60  0000 C CNN
+F 3 "" H 5250 2500 60  0000 C CNN
+F 4 "TPS73001DBVR" H 5250 2500 60  0001 C CNN "MPN"
+	1    5250 2500
+	1    0    0    -1
+$EndComp
+$Comp
+L TPS73001 U4
+U 1 1 5494586A
+P 5250 4050
+F 0 "U4" H 5200 4300 60  0000 C CNN
+F 1 "TPS73001" H 5500 3800 60  0000 C CNN
+F 2 "" H 5250 4050 60  0000 C CNN
+F 3 "" H 5250 4050 60  0000 C CNN
+	1    5250 4050
+	1    0    0    -1
+$EndComp
 $EndSCHEMATC

Commit message: whole bunch of stuff
Parts:
- C17, C21, C26, C27: footprint (none) -> Capacitors_SMD:C_0603
- C18, C19, C20, C22, C23, C24, C25: footprint (none) -> Capacitors_SMD:C_0402
- SW1: MPN (none) -> PTS840 GM SMTR LFS
Other:
- note added: "Turn stuff on"
Changed lines of the file:
@@
 F 0 "C20" H 4000 2700 50  0000 L CNN
 F 1 "1uF" H 4000 2500 50  0000 L CNN
-F 2 "" H 3950 2600 60  0000 C CNN
+F 2 "Capacitors_SMD:C_0402" H 3950 2600 60  0001 C CNN
 F 3 "" H 3950 2600 60  0000 C CNN
 	1    3950 2600
@@
 F 0 "BT1" H 6850 6350 50  0000 C CNN
 F 1 "BATTERY" H 6850 5960 50  0000 C CNN
-F 2 "" H 6850 6150 60  0000 C CNN
+F 2 "" H 6850 6150 60  0001 C CNN
 F 3 "" H 6850 6150 60  0000 C CNN
 	1    6850 6150
@@
 F 0 "C22" H 4750 3400 50  0000 L CNN
 F 1 "10nF" H 4750 3200 50  0000 L CNN
-F 2 "" H 4700 3300 60  0000 C CNN
+F 2 "Capacitors_SMD:C_0402" H 4700 3300 60  0001 C CNN
 F 3 "" H 4700 3300 60  0000 C CNN
 	1    4700 3300
@@
 F 0 "C26" H 7050 2700 50  0000 L CNN
 F 1 "4.7uF" H 7050 2500 50  0000 L CNN
-F 2 "" H 7000 2600 60  0000 C CNN
+F 2 "Capacitors_SMD:C_0603" H 7000 2600 60  0001 C CNN
 F 3 "" H 7000 2600 60  0000 C CNN
 F 4 "CL10B475KQ8NQNC" H 7000 2600 60  0001 C CNN "MPN"
@@
 F 0 "R14" V 5630 3200 50  0000 C CNN
 F 1 "0" V 5550 3200 50  0000 C CNN
-F 2 "" H 5550 3200 60  0000 C CNN
+F 2 "" H 5550 3200 60  0001 C CNN
 F 3 "" H 5550 3200 60  0000 C CNN
 F 4 "RC1005J000CS" V 5550 3200 60  0001 C CNN "MPN"
@@
 F 0 "R16" V 6280 2650 50  0000 C CNN
 F 1 "39k" V 6200 2650 50  0000 C CNN
-F 2 "" H 6200 2650 60  0000 C CNN
+F 2 "" H 6200 2650 60  0001 C CNN
 F 3 "" H 6200 2650 60  0000 C CNN
 F 4 "RC1005J393CS" V 6200 2650 60  0001 C CNN "MPN"
@@
 F 0 "R17" V 6280 3250 50  0000 C CNN
 F 1 "30k" V 6200 3250 50  0000 C CNN
-F 2 "" H 6200 3250 60  0000 C CNN
+F 2 "" H 6200 3250 60  0001 C CNN
 F 3 "" H 6200 3250 60  0000 C CNN
 F 4 "RC1005J303CS" V 6200 3250 60  0001 C CNN "MPN"
@@
 F 0 "C24" H 6550 2750 50  0000 L CNN
 F 1 "22pF" H 6550 2550 50  0000 L CNN
-F 2 "" H 6500 2650 60  0000 C CNN
+F 2 "Capacitors_SMD:C_0402" H 6500 2650 60  0001 C CNN
 F 3 "" H 6500 2650 60  0000 C CNN
 F 4 "CL05C220JB5NNNC" H 6500 2650 60  0001 C CNN "MPN"
@@
 F 0 "C21" H 4000 4250 50  0000 L CNN
 F 1 "4.7uF" H 4000 4050 50  0000 L CNN
-F 2 "" H 3950 4150 60  0000 C CNN
+F 2 "Capacitors_SMD:C_0603" H 3950 4150 60  0001 C CNN
 F 3 "" H 3950 4150 60  0000 C CNN
 	1    3950 4150
@@
 F 0 "C23" H 4750 4950 50  0000 L CNN
 F 1 "10nF" H 4750 4750 50  0000 L CNN
-F 2 "" H 4700 4850 60  0000 C CNN
+F 2 "Capacitors_SMD:C_0402" H 4700 4850 60  0001 C CNN
 F 3 "" H 4700 4850 60  0000 C CNN
 	1    4700 4850
@@
 F 0 "C27" H 7050 4250 50  0000 L CNN
 F 1 "4.7uF" H 7050 4050 50  0000 L CNN
-F 2 "" H 7000 4150 60  0000 C CNN
+F 2 "Capacitors_SMD:C_0603" H 7000 4150 60  0001 C CNN
 F 3 "" H 7000 4150 60  0000 C CNN
 	1    7000 4150
@@
 F 0 "R15" V 5630 4750 50  0000 C CNN
 F 1 "0" V 5550 4750 50  0000 C CNN
-F 2 "" H 5550 4750 60  0000 C CNN
+F 2 "" H 5550 4750 60  0001 C CNN
 F 3 "" H 5550 4750 60  0000 C CNN
 	1    5550 4750
@@
 F 0 "R18" V 6280 4200 50  0000 C CNN
 F 1 "39k" V 6200 4200 50  0000 C CNN
-F 2 "" H 6200 4200 60  0000 C CNN
+F 2 "" H 6200 4200 60  0001 C CNN
 F 3 "" H 6200 4200 60  0000 C CNN
 	1    6200 4200
@@
 F 0 "R19" V 6280 4800 50  0000 C CNN
 F 1 "30k" V 6200 4800 50  0000 C CNN
-F 2 "" H 6200 4800 60  0000 C CNN
+F 2 "" H 6200 4800 60  0001 C CNN
 F 3 "" H 6200 4800 60  0000 C CNN
 	1    6200 4800
@@
 F 0 "C25" H 6550 4300 50  0000 L CNN
 F 1 "22pF" H 6550 4100 50  0000 L CNN
-F 2 "" H 6500 4200 60  0000 C CNN
+F 2 "Capacitors_SMD:C_0402" H 6500 4200 60  0001 C CNN
 F 3 "" H 6500 4200 60  0000 C CNN
 	1    6500 4200
@@
 F 0 "R11" V 3630 3950 50  0000 C CNN
 F 1 "10" V 3550 3950 50  0000 C CNN
-F 2 "" H 3550 3950 60  0000 C CNN
+F 2 "" H 3550 3950 60  0001 C CNN
 F 3 "" H 3550 3950 60  0000 C CNN
 F 4 "MCR01MRTF10R0" V 3550 3950 60  0001 C CNN "MPN"
@@
 F 0 "C17" H 2850 4250 50  0000 L CNN
 F 1 "4.7uF" H 2850 4050 50  0000 L CNN
-F 2 "" H 2800 4150 60  0000 C CNN
+F 2 "Capacitors_SMD:C_0603" H 2800 4150 60  0001 C CNN
 F 3 "" H 2800 4150 60  0000 C CNN
 	1    2800 4150
@@
 F 0 "C18" H 3200 4250 50  0000 L CNN
 F 1 "100nF" H 3200 4050 50  0000 L CNN
-F 2 "" H 3150 4150 60  0000 C CNN
+F 2 "Capacitors_SMD:C_0402" H 3150 4150 60  0001 C CNN
 F 3 "" H 3150 4150 60  0000 C CNN
 	1    3150 4150
@@
 F 0 "SW1" H 1900 6360 50  0000 C CNN
 F 1 "SW_PUSH" H 1750 6170 50  0000 C CNN
-F 2 "" H 1750 6250 60  0000 C CNN
+F 2 "" H 1750 6250 60  0001 C CNN
 F 3 "" H 1750 6250 60  0000 C CNN
+F 4 "PTS840 GM SMTR LFS" H 1750 6250 60  0001 C CNN "MPN"
 	1    1750 6250
 	1    0    0    -1
@@
 F 0 "R10" V 2930 6500 50  0000 C CNN
 F 1 "100k" V 2850 6500 50  0000 C CNN
-F 2 "" H 2850 6500 60  0000 C CNN
+F 2 "" H 2850 6500 60  0001 C CNN
 F 3 "" H 2850 6500 60  0000 C CNN
 F 4 "MCR01MRTF1003" V 2850 6500 60  0001 C CNN "MPN"
@@
 F 0 "D2" H 2150 7150 50  0000 C CNN
 F 1 "2.7v" H 2150 6950 40  0000 C CNN
-F 2 "" H 2150 7050 60  0000 C CNN
+F 2 "" H 2150 7050 60  0001 C CNN
 F 3 "" H 2150 7050 60  0000 C CNN
 F 4 "MM3Z2V7T1G" H 2150 7050 60  0001 C CNN "MPN"
@@
 F 0 "R8" V 2230 6500 50  0000 C CNN
 F 1 "2k2" V 2150 6500 50  0000 C CNN
-F 2 "" H 2150 6500 60  0000 C CNN
+F 2 "" H 2150 6500 60  0001 C CNN
 F 3 "" H 2150 6500 60  0000 C CNN
 F 4 "RMCF0402JT2K20" V 2150 6500 60  0001 C CNN "MPN"
@@
 F 0 "C19" H 3200 6550 50  0000 L CNN
 F 1 "10nF" H 3200 6350 50  0000 L CNN
-F 2 "" H 3150 6450 60  0000 C CNN
+F 2 "Capacitors_SMD:C_0402" H 3150 6450 60  0001 C CNN
 F 3 "" H 3150 6450 60  0000 C CNN
 	1    3150 6450
@@
 F 0 "R9" V 2530 7050 50  0000 C CNN
 F 1 "20k" V 2450 7050 50  0000 C CNN
-F 2 "" H 2450 7050 60  0000 C CNN
+F 2 "" H 2450 7050 60  0001 C CNN
 F 3 "" H 2450 7050 60  0000 C CNN
 F 4 "MCR01MRTF2002" V 2450 7050 60  0001 C CNN "MPN"
@@
 F 0 "R13" V 5380 6850 50  0000 C CNN
 F 1 "62k" V 5300 6850 50  0000 C CNN
-F 2 "" H 5300 6850 60  0000 C CNN
+F 2 "" H 5300 6850 60  0001 C CNN
 F 3 "" H 5300 6850 60  0000 C CNN
 F 4 "MCR01MRTJ623" V 5300 6850 60  0001 C CNN "MPN"
@@
 F 0 "R12" V 5380 6250 50  0000 C CNN
 F 1 "36k" V 5300 6250 50  0000 C CNN
-F 2 "" H 5300 6250 60  0000 C CNN
+F 2 "" H 5300 6250 60  0001 C CNN
 F 3 "" H 5300 6250 60  0000 C CNN
 F 4 "MCR01MRTF3602" V 5300 6250 60  0001 C CNN "MPN"
@@
 F 0 "D3" H 2500 6350 40  0000 C CNN
 F 1 "BAT54C" H 2500 5950 40  0000 C CNN
-F 2 "" H 2500 6300 60  0000 C CNN
+F 2 "" H 2500 6300 60  0001 C CNN
 F 3 "" H 2500 6300 60  0000 C CNN
 	1    2500 6150
@@
 F 0 "U3" H 5200 2750 60  0000 C CNN
 F 1 "TPS73001" H 5500 2250 60  0000 C CNN
-F 2 "" H 5250 2500 60  0000 C CNN
+F 2 "" H 5250 2500 60  0001 C CNN
 F 3 "" H 5250 2500 60  0000 C CNN
 F 4 "TPS73001DBVR" H 5250 2500 60  0001 C CNN "MPN"
@@
 F 0 "U4" H 5200 4300 60  0000 C CNN
 F 1 "TPS73001" H 5500 3800 60  0000 C CNN
-F 2 "" H 5250 4050 60  0000 C CNN
+F 2 "" H 5250 4050 60  0001 C CNN
 F 3 "" H 5250 4050 60  0000 C CNN
 	1    5250 4050
 	1    0    0    -1
 $EndComp
+Text Notes 2450 5800 0    60   ~ 0
+Turn stuff on
 $EndSCHEMATC

Commit message: more stuff
Parts:
- D3: footprint (none) -> Diodes_SMD:Diode_SOT23
Changed lines of the file:
@@
 F 0 "D3" H 2500 6350 40  0000 C CNN
 F 1 "BAT54C" H 2500 5950 40  0000 C CNN
-F 2 "" H 2500 6300 60  0001 C CNN
+F 2 "Diodes_SMD:Diode_SOT23" H 2500 6300 60  0001 C CNN
 F 3 "" H 2500 6300 60  0000 C CNN
 	1    2500 6150
