File: cad/sensors.sch (KiCad schematic (older format))
At the start: 4 parts

Commit message: passed erc
Parts:
- gave numbers to parts that had none: 4
Changed lines of the file:
@@
 $EndDescr
 $Comp
-L MPU-9250 U?
+L MPU-9250 U2
 U 1 1 548C98CF
 P 5600 3750
-F 0 "U?" H 5600 4450 60  0000 C CNN
+F 0 "U2" H 5600 4450 60  0000 C CNN
 F 1 "MPU-9250" H 5600 3050 60  0000 C CNN
 F 2 "" H 5700 3850 60  0000 C CNN
@@
 $EndComp
 $Comp
-L C C?
+L C C16
 U 1 1 548D972B
 P 4600 4500
-F 0 "C?" H 4650 4600 50  0000 L CNN
+F 0 "C16" H 4650 4600 50  0000 L CNN
 F 1 "10nF" H 4650 4400 50  0000 L CNN
 F 2 "" H 4600 4500 60  0000 C CNN
@@
 $EndComp
 $Comp
-L C C?
+L C C15
 U 1 1 548D97BB
 P 4150 4500
-F 0 "C?" H 4200 4600 50  0000 L CNN
+F 0 "C15" H 4200 4600 50  0000 L CNN
 F 1 "100nF" H 4200 4400 50  0000 L CNN
 F 2 "" H 4150 4500 60  0000 C CNN
@@
 $EndComp
 $Comp
-L C C?
+L C C14
 U 1 1 548D9E9A
 P 3250 4150
-F 0 "C?" H 3300 4250 50  0000 L CNN
+F 0 "C14" H 3300 4250 50  0000 L CNN
 F 1 "100nF" H 3300 4050 50  0000 L CNN
 F 2 "" H 3250 4150 60  0000 C CNN

Commit message: selecting parts for the little passives
Parts:
- C16: MPN (none) -> GRM155R71E103KA01D
- U2: MPN (none) -> MPU-9250
Changed lines of the file:
@@
 F 2 "" H 5700 3850 60  0000 C CNN
 F 3 "" H 5700 3850 60  0000 C CNN
+F 4 "MPU-9250" H 5600 3750 60  0001 C CNN "MPN"
 	1    5600 3750
 	1    0    0    -1
@@
 F 2 "" H 4600 4500 60  0000 C CNN
 F 3 "" H 4600 4500 60  0000 C CNN
+F 4 "GRM155R71E103KA01D" H 4600 4500 60  0001 C CNN "MPN"
 	1    4600 4500
 	1    0    0    -1

Commit message: whole bunch of stuff
Parts:
- C14, C15, C16: footprint (none) -> Capacitors_SMD:C_0402
Changed lines of the file:
@@
 F 0 "U2" H 5600 4450 60  0000 C CNN
 F 1 "MPU-9250" H 5600 3050 60  0000 C CNN
-F 2 "" H 5700 3850 60  0000 C CNN
+F 2 "" H 5700 3850 60  0001 C CNN
 F 3 "" H 5700 3850 60  0000 C CNN
 F 4 "MPU-9250" H 5600 3750 60  0001 C CNN "MPN"
@@
 F 0 "C16" H 4650 4600 50  0000 L CNN
 F 1 "10nF" H 4650 4400 50  0000 L CNN
-F 2 "" H 4600 4500 60  0000 C CNN
+F 2 "Capacitors_SMD:C_0402" H 4600 4500 60  0001 C CNN
 F 3 "" H 4600 4500 60  0000 C CNN
 F 4 "GRM155R71E103KA01D" H 4600 4500 60  0001 C CNN "MPN"
@@
 F 0 "C15" H 4200 4600 50  0000 L CNN
 F 1 "100nF" H 4200 4400 50  0000 L CNN
-F 2 "" H 4150 4500 60  0000 C CNN
+F 2 "Capacitors_SMD:C_0402" H 4150 4500 60  0001 C CNN
 F 3 "" H 4150 4500 60  0000 C CNN
 	1    4150 4500
@@
 F 0 "C14" H 3300 4250 50  0000 L CNN
 F 1 "100nF" H 3300 4050 50  0000 L CNN
-F 2 "" H 3250 4150 60  0000 C CNN
+F 2 "Capacitors_SMD:C_0402" H 3250 4150 60  0001 C CNN
 F 3 "" H 3250 4150 60  0000 C CNN
 	1    3250 4150

Commit message: bunch more footprints assigned
Parts:
- U2: footprint (none) -> SMD_Packages:QFN-28-1EP
Changed lines of the file:
@@
 F 0 "U2" H 5600 4450 60  0000 C CNN
 F 1 "MPU-9250" H 5600 3050 60  0000 C CNN
-F 2 "" H 5700 3850 60  0001 C CNN
+F 2 "SMD_Packages:QFN-28-1EP" H 5700 3850 60  0001 C CNN
 F 3 "" H 5700 3850 60  0000 C CNN
 F 4 "MPU-9250" H 5600 3750 60  0001 C CNN "MPN"
