File: cad/smartercopter.sch (KiCad schematic (older format))
At the start: 26 parts, among them P1 CONN_5, U1 CC2541, X1 32Mhz

Commit message: selecting parts for the little passives
Parts:
- C7: MPN (none) -> CC0402KRX7R9BB221
- C9: MPN (none) -> GRM155R71H102KA01D
- R1: MPN (none) -> 1-1622826-8
- R3: MPN (none) -> RMCF0402JT2K70
- R6: MPN (none) -> MCR01MRTF5602
- U1: MPN (none) -> CC2541F256RHAR
Changed lines of the file:
@@
 F 2 "" H 4500 1250 60  0000 C CNN
 F 3 "" H 4500 1250 60  0000 C CNN
+F 4 "CC2541F256RHAR" H 4100 2650 60  0001 C CNN "MPN"
 	1    4100 2650
 	1    0    0    -1
@@
 F 2 "" H 5438 3050 30  0000 C CNN
 F 3 "" H 5400 3200 60  0000 C CNN
+F 4 "GRM155R71H102KA01D" H 5400 3200 60  0001 C CNN "MPN"
 	1    5400 3200
 	1    0    0    -1
@@
 F 2 "" V 5730 3000 30  0000 C CNN
 F 3 "" H 5800 3000 30  0000 C CNN
+F 4 "RMCF0402JT2K70" V 5800 3000 60  0001 C CNN "MPN"
 	1    5800 3000
 	0    1    1    0
@@
 F 2 "" V 6630 2800 30  0000 C CNN
 F 3 "" H 6700 2800 30  0000 C CNN
+F 4 "MCR01MRTF5602" V 6700 2800 60  0001 C CNN "MPN"
 	1    6700 2800
 	0    1    1    0
@@
 F 2 "" H 3750 5450 60  0000 C CNN
 F 3 "" H 3750 5450 60  0000 C CNN
+F 4 "CC0402KRX7R9BB221" H 3750 5450 60  0001 C CNN "MPN"
 	1    3750 5450
 	1    0    0    -1
@@
 F 2 "" V 2180 6350 30  0000 C CNN
 F 3 "" H 2250 6350 30  0000 C CNN
+F 4 "1-1622826-8" V 2250 6350 60  0001 C CNN "MPN"
 	1    2250 6350
 	0    1    1    0

Commit message: whole bunch of stuff
Parts:
- removed D1: BI_LED, symbol BI_LED
- added D1: BI_COLOR_LED, symbol BI_COLOR_LED
- C1, C12, C13, C2, C3, C4, C5, C6, C7, C8, C9: footprint (none) -> Capacitors_SMD:C_0402
- C10, C11: footprint (none) -> Capacitors_SMD:C_0201
- X1: MPN FA-128 32MHz 10pF 10PPM -> FA-128 32.0000MF20X-K3
Connections:
- wire segments 101 -> 104
Other:
- moved on the sheet: R2
Changed lines of the file:
@@
 F 0 "U1" H 3650 4150 60  0000 C CNN
 F 1 "CC2541" H 3750 1000 60  0000 C CNN
-F 2 "" H 4500 1250 60  0000 C CNN
+F 2 "" H 4500 1250 60  0001 C CNN
 F 3 "" H 4500 1250 60  0000 C CNN
 F 4 "CC2541F256RHAR" H 4100 2650 60  0001 C CNN "MPN"
@@
 F 0 "C8" H 5100 4000 40  0000 L CNN
 F 1 "1uF" H 5106 3815 40  0000 L CNN
-F 2 "" H 5138 3750 30  0000 C CNN
+F 2 "Capacitors_SMD:C_0402" H 5138 3750 30  0001 C CNN
 F 3 "" H 5100 3900 60  0000 C CNN
 	1    5100 3900
@@
 F 0 "C9" H 5400 3300 40  0000 L CNN
 F 1 "1nF" H 5406 3115 40  0000 L CNN
-F 2 "" H 5438 3050 30  0000 C CNN
+F 2 "Capacitors_SMD:C_0402" H 5438 3050 30  0001 C CNN
 F 3 "" H 5400 3200 60  0000 C CNN
 F 4 "GRM155R71H102KA01D" H 5400 3200 60  0001 C CNN "MPN"
@@
 F 0 "R3" V 5880 3000 40  0000 C CNN
 F 1 "2k7" V 5807 3001 40  0000 C CNN
-F 2 "" V 5730 3000 30  0000 C CNN
+F 2 "" V 5730 3000 30  0001 C CNN
 F 3 "" H 5800 3000 30  0000 C CNN
 F 4 "RMCF0402JT2K70" V 5800 3000 60  0001 C CNN "MPN"
@@
 F 0 "R6" V 6780 2800 40  0000 C CNN
 F 1 "56k" V 6707 2801 40  0000 C CNN
-F 2 "" V 6630 2800 30  0000 C CNN
+F 2 "" V 6630 2800 30  0001 C CNN
 F 3 "" H 6700 2800 30  0000 C CNN
 F 4 "MCR01MRTF5602" V 6700 2800 60  0001 C CNN "MPN"
@@
 F 0 "C11" H 6850 4150 50  0000 L CNN
 F 1 "12pF" H 6850 3950 50  0000 L CNN
-F 2 "" H 6800 4050 60  0000 C CNN
+F 2 "Capacitors_SMD:C_0201" H 6800 4050 60  0001 C CNN
 F 3 "" H 6800 4050 60  0000 C CNN
 	1    6800 4050
@@
 F 0 "C10" H 6250 4150 50  0000 L CNN
 F 1 "12pF" H 6250 3950 50  0000 L CNN
-F 2 "" H 6200 4050 60  0000 C CNN
+F 2 "Capacitors_SMD:C_0201" H 6200 4050 60  0001 C CNN
 F 3 "" H 6200 4050 60  0000 C CNN
 F 4 "02013A120JAT2A" H 6200 4050 60  0001 C CNN "MPN"
@@
 F 0 "C1" H 1800 5550 50  0000 L CNN
 F 1 "1uF" H 1800 5350 50  0000 L CNN
-F 2 "" H 1750 5450 60  0000 C CNN
+F 2 "Capacitors_SMD:C_0402" H 1750 5450 60  0001 C CNN
 F 3 "" H 1750 5450 60  0000 C CNN
 F 4 "GRM155R60J105KE19D" H 1750 5450 60  0001 C CNN "MPN"
@@
 F 0 "C2" H 2050 5550 50  0000 L CNN
 F 1 "100nF" H 2050 5350 50  0000 L CNN
-F 2 "" H 2000 5450 60  0000 C CNN
+F 2 "Capacitors_SMD:C_0402" H 2000 5450 60  0001 C CNN
 F 3 "" H 2000 5450 60  0000 C CNN
 F 4 "LMK105BJ104KV-F" H 2000 5450 60  0001 C CNN "MPN"
@@
 F 0 "C3" H 2400 5550 50  0000 L CNN
 F 1 "100nF" H 2400 5350 50  0000 L CNN
-F 2 "" H 2350 5450 60  0000 C CNN
+F 2 "Capacitors_SMD:C_0402" H 2350 5450 60  0001 C CNN
 F 3 "" H 2350 5450 60  0000 C CNN
 	1    2350 5450
@@
 F 0 "C4" H 2750 5550 50  0000 L CNN
 F 1 "100nF" H 2750 5350 50  0000 L CNN
-F 2 "" H 2700 5450 60  0000 C CNN
+F 2 "Capacitors_SMD:C_0402" H 2700 5450 60  0001 C CNN
 F 3 "" H 2700 5450 60  0000 C CNN
 	1    2700 5450
@@
 F 0 "C5" H 3100 5550 50  0000 L CNN
 F 1 "100nF" H 3100 5350 50  0000 L CNN
-F 2 "" H 3050 5450 60  0000 C CNN
+F 2 "Capacitors_SMD:C_0402" H 3050 5450 60  0001 C CNN
 F 3 "" H 3050 5450 60  0000 C CNN
 	1    3050 5450
@@
 F 0 "C6" H 3450 5550 50  0000 L CNN
 F 1 "100nF" H 3450 5350 50  0000 L CNN
-F 2 "" H 3400 5450 60  0000 C CNN
+F 2 "Capacitors_SMD:C_0402" H 3400 5450 60  0001 C CNN
 F 3 "" H 3400 5450 60  0000 C CNN
 	1    3400 5450
@@
 F 0 "C7" H 3800 5550 50  0000 L CNN
 F 1 "220pF" H 3800 5350 50  0000 L CNN
-F 2 "" H 3750 5450 60  0000 C CNN
+F 2 "Capacitors_SMD:C_0402" H 3750 5450 60  0001 C CNN
 F 3 "" H 3750 5450 60  0000 C CNN
 F 4 "CC0402KRX7R9BB221" H 3750 5450 60  0001 C CNN "MPN"
@@
 F 0 "R4" V 6030 1800 40  0000 C CNN
 F 1 "2k2" V 5957 1801 40  0000 C CNN
-F 2 "" V 5880 1800 30  0000 C CNN
+F 2 "" V 5880 1800 30  0001 C CNN
 F 3 "" H 5950 1800 30  0000 C CNN
 	1    5950 1800
@@
 F 0 "R5" V 6230 1800 40  0000 C CNN
 F 1 "2k2" V 6157 1801 40  0000 C CNN
-F 2 "" V 6080 1800 30  0000 C CNN
+F 2 "" V 6080 1800 30  0001 C CNN
 F 3 "" H 6150 1800 30  0000 C CNN
 	1    6150 1800
@@
 F 0 "X1" H 6500 4000 30  0000 C CNN
 F 1 "32Mhz" H 6300 3950 30  0000 L CNN
-F 2 "" H 6500 3850 60  0000 C CNN
+F 2 "" H 6500 3850 60  0001 C CNN
 F 3 "" H 6500 3850 60  0000 C CNN
-F 4 "FA-128 32MHz 10pF 10PPM" H 6500 3850 60  0001 C CNN "MPN"
+F 4 "FA-128 32.0000MF20X-K3" H 6500 3850 60  0001 C CNN "MPN"
 	1    6500 3850
 	1    0    0    -1
@@
 F 0 "FL1" H 8450 5800 60  0000 C CNN
 F 1 "2450BM15A0002" H 8450 5300 60  0000 C CNN
-F 2 "" H 8500 5350 60  0000 C CNN
+F 2 "" H 8500 5350 60  0001 C CNN
 F 3 "" H 8500 5350 60  0000 C CNN
 F 4 "2450BM15A0002" H 8400 5550 60  0001 C CNN "MPN"
@@
 F 0 "A1" H 9950 6450 60  0000 C CNN
 F 1 "2450AT42A100" H 9950 5950 60  0000 C CNN
-F 2 "" H 9950 6050 60  0000 C CNN
+F 2 "" H 9950 6050 60  0001 C CNN
 F 3 "" H 9950 6050 60  0000 C CNN
 F 4 "2450AT42A100" H 9950 6050 60  0001 C CNN "MPN"
@@
 F 0 "C12" H 8700 6350 40  0000 L CNN
 F 1 "DNM" H 8706 6165 40  0000 L CNN
-F 2 "" H 8738 6100 30  0000 C CNN
+F 2 "Capacitors_SMD:C_0402" H 8738 6100 30  0001 C CNN
 F 3 "" H 8700 6250 60  0000 C CNN
 	1    8700 6250
@@
 F 0 "C13" H 9400 6350 40  0000 L CNN
 F 1 "DNM" H 9406 6165 40  0000 L CNN
-F 2 "" H 9438 6100 30  0000 C CNN
+F 2 "Capacitors_SMD:C_0402" H 9438 6100 30  0001 C CNN
 F 3 "" H 9400 6250 60  0000 C CNN
 	1    9400 6250
@@
 F 0 "R7" V 9130 6050 40  0000 C CNN
 F 1 "0" V 9057 6051 40  0000 C CNN
-F 2 "" V 8980 6050 30  0000 C CNN
+F 2 "" V 8980 6050 30  0001 C CNN
 F 3 "" H 9050 6050 30  0000 C CNN
 	1    9050 6050
@@
 F 0 "R1" V 2330 6350 40  0000 C CNN
 F 1 "1K" V 2257 6351 40  0000 C CNN
-F 2 "" V 2180 6350 30  0000 C CNN
+F 2 "" V 2180 6350 30  0001 C CNN
 F 3 "" H 2250 6350 30  0000 C CNN
 F 4 "1-1622826-8" V 2250 6350 60  0001 C CNN "MPN"
@@
 $EndComp
 $Comp
-L BI_LED D1
-U 1 1 549157A0
-P 2800 6450
-F 0 "D1" H 3100 6550 50  0000 C CNN
-F 1 "BI_LED" H 3150 6350 50  0000 C CNN
-F 2 "" H 2800 6450 60  0000 C CNN
-F 3 "" H 2800 6450 60  0000 C CNN
-	1    2800 6450
-	1    0    0    -1
-$EndComp
-$Comp
 L R R2
 U 1 1 54915854
-P 2250 6550
-F 0 "R2" V 2330 6550 40  0000 C CNN
-F 1 "1K" V 2257 6551 40  0000 C CNN
-F 2 "" V 2180 6550 30  0000 C CNN
-F 3 "" H 2250 6550 30  0000 C CNN
-	1    2250 6550
+P 2250 6700
+F 0 "R2" V 2330 6700 40  0000 C CNN
+F 1 "1K" V 2257 6701 40  0000 C CNN
+F 2 "" V 2180 6700 30  0001 C CNN
+F 3 "" H 2250 6700 30  0000 C CNN
+	1    2250 6700
 	0    1    1    0
 $EndComp
@@
 L DGND #PWR022
 U 1 1 549158BD
-P 3350 6650
-F 0 "#PWR022" H 3350 6650 40  0001 C CNN
-F 1 "DGND" H 3350 6580 40  0000 C CNN
-F 2 "" H 3350 6650 60  0000 C CNN
-F 3 "" H 3350 6650 60  0000 C CNN
-	1    3350 6650
-	1    0    0    -1
-$EndComp
-Wire Wire Line
-	3150 6450 3350 6450
-Wire Wire Line
-	3350 6450 3350 6650
+P 3350 6750
+F 0 "#PWR022" H 3350 6750 40  0001 C CNN
+F 1 "DGND" H 3350 6680 40  0000 C CNN
+F 2 "" H 3350 6750 60  0000 C CNN
+F 3 "" H 3350 6750 60  0000 C CNN
+	1    3350 6750
+	1    0    0    -1
+$EndComp
+Wire Wire Line
+	3150 6550 3350 6550
+Wire Wire Line
+	3350 6550 3350 6750
 Wire Wire Line
 	2000 6350 1650 6350
 Wire Wire Line
-	2000 6550 1650 6550
+	2000 6700 1650 6700
 Text Label 1650 6350 0    60   ~ 0
 LED1
-Text Label 1650 6550 0    60   ~ 0
+Text Label 1650 6700 0    60   ~ 0
 LED2
 $Comp
@@
 F 0 "P1" H 5900 5650 50  0000 C CNN
 F 1 "CONN_5" V 6000 5350 50  0000 C CNN
-F 2 "" H 5900 5350 60  0000 C CNN
+F 2 "" H 5900 5350 60  0001 C CNN
 F 3 "" H 5900 5350 60  0000 C CNN
 	1    5900 5350
@@
 NoConn ~ 3350 2800
 NoConn ~ 3350 2900
+$Comp
+L BI_COLOR_LED D1
+U 1 1 54952C6A
+P 2700 6350
+F 0 "D1" H 2700 6450 50  0000 C CNN
+F 1 "BI_COLOR_LED" H 2700 6250 50  0000 C CNN
+F 2 "" H 2700 6350 60  0001 C CNN
+F 3 "" H 2700 6350 60  0000 C CNN
+F 4 "APTB1612ESGC-F01" H 2700 6350 60  0001 C CNN "MPN"
+	1    2700 6350
+	1    0    0    -1
+$EndComp
+$Comp
+L BI_COLOR_LED D1
+U 2 1 54952CD6
+P 2700 6700
+F 0 "D1" H 2700 6800 50  0000 C CNN
+F 1 "BI_COLOR_LED" H 2700 6600 50  0000 C CNN
+F 2 "" H 2700 6700 60  0001 C CNN
+F 3 "" H 2700 6700 60  0000 C CNN
+	2    2700 6700
+	1    0    0    -1
+$EndComp
+Wire Wire Line
+	2900 6350 3150 6350
+Wire Wire Line
+	3150 6350 3150 6700
+Wire Wire Line
+	3150 6700 2900 6700
+Connection ~ 3150 6550
 $EndSCHEMATC

Commit message: added more footprint stuff
Parts:
- R1, R2, R3, R4, R5, R6, R7: footprint (none) -> Resistors_SMD:R_0402
Changed lines of the file:
@@
 LIBS:valves
 LIBS:misc
-LIBS:MPU-9250
-LIBS:p8x32a-lqfp
-LIBS:cc2541
 LIBS:device
 LIBS:smartercopter-cache
@@
 F 0 "R3" V 5880 3000 40  0000 C CNN
 F 1 "2k7" V 5807 3001 40  0000 C CNN
-F 2 "" V 5730 3000 30  0001 C CNN
+F 2 "Resistors_SMD:R_0402" V 5730 3000 30  0001 C CNN
 F 3 "" H 5800 3000 30  0000 C CNN
 F 4 "RMCF0402JT2K70" V 5800 3000 60  0001 C CNN "MPN"
@@
 F 0 "R6" V 6780 2800 40  0000 C CNN
 F 1 "56k" V 6707 2801 40  0000 C CNN
-F 2 "" V 6630 2800 30  0001 C CNN
+F 2 "Resistors_SMD:R_0402" V 6630 2800 30  0001 C CNN
 F 3 "" H 6700 2800 30  0000 C CNN
 F 4 "MCR01MRTF5602" V 6700 2800 60  0001 C CNN "MPN"
@@
 F 0 "R4" V 6030 1800 40  0000 C CNN
 F 1 "2k2" V 5957 1801 40  0000 C CNN
-F 2 "" V 5880 1800 30  0001 C CNN
+F 2 "Resistors_SMD:R_0402" V 5880 1800 30  0001 C CNN
 F 3 "" H 5950 1800 30  0000 C CNN
 	1    5950 1800
@@
 F 0 "R5" V 6230 1800 40  0000 C CNN
 F 1 "2k2" V 6157 1801 40  0000 C CNN
-F 2 "" V 6080 1800 30  0001 C CNN
+F 2 "Resistors_SMD:R_0402" V 6080 1800 30  0001 C CNN
 F 3 "" H 6150 1800 30  0000 C CNN
 	1    6150 1800
@@
 F 0 "R7" V 9130 6050 40  0000 C CNN
 F 1 "0" V 9057 6051 40  0000 C CNN
-F 2 "" V 8980 6050 30  0001 C CNN
+F 2 "Resistors_SMD:R_0402" V 8980 6050 30  0001 C CNN
 F 3 "" H 9050 6050 30  0000 C CNN
 	1    9050 6050
@@
 F 0 "R1" V 2330 6350 40  0000 C CNN
 F 1 "1K" V 2257 6351 40  0000 C CNN
-F 2 "" V 2180 6350 30  0001 C CNN
+F 2 "Resistors_SMD:R_0402" V 2180 6350 30  0001 C CNN
 F 3 "" H 2250 6350 30  0000 C CNN
 F 4 "1-1622826-8" V 2250 6350 60  0001 C CNN "MPN"
@@
 F 0 "R2" V 2330 6700 40  0000 C CNN
 F 1 "1K" V 2257 6701 40  0000 C CNN
-F 2 "" V 2180 6700 30  0001 C CNN
+F 2 "Resistors_SMD:R_0402" V 2180 6700 30  0001 C CNN
 F 3 "" H 2250 6700 30  0000 C CNN
 	1    2250 6700

Commit message: bunch more footprints assigned
Parts:
- A1: footprint (none) -> hlib:2450AT42A100
- D1: footprint (none) -> hlib:APTB1612ESGC-F01
- FL1: footprint (none) -> hlib:2450BM15A0002
- U1: footprint (none) -> SMD_Packages:LFCSP-40-1EP
- X1: footprint (none) -> hlib:4-SMD
Changed lines of the file:
@@
 F 0 "U1" H 3650 4150 60  0000 C CNN
 F 1 "CC2541" H 3750 1000 60  0000 C CNN
-F 2 "" H 4500 1250 60  0001 C CNN
+F 2 "SMD_Packages:LFCSP-40-1EP" H 4500 1250 60  0001 C CNN
 F 3 "" H 4500 1250 60  0000 C CNN
 F 4 "CC2541F256RHAR" H 4100 2650 60  0001 C CNN "MPN"
@@
 F 0 "X1" H 6500 4000 30  0000 C CNN
 F 1 "32Mhz" H 6300 3950 30  0000 L CNN
-F 2 "" H 6500 3850 60  0001 C CNN
+F 2 "hlib:4-SMD" H 6500 3850 60  0001 C CNN
 F 3 "" H 6500 3850 60  0000 C CNN
 F 4 "FA-128 32.0000MF20X-K3" H 6500 3850 60  0001 C CNN "MPN"
@@
 F 0 "FL1" H 8450 5800 60  0000 C CNN
 F 1 "2450BM15A0002" H 8450 5300 60  0000 C CNN
-F 2 "" H 8500 5350 60  0001 C CNN
+F 2 "hlib:2450BM15A0002" H 8500 5350 60  0001 C CNN
 F 3 "" H 8500 5350 60  0000 C CNN
 F 4 "2450BM15A0002" H 8400 5550 60  0001 C CNN "MPN"
@@
 F 0 "A1" H 9950 6450 60  0000 C CNN
 F 1 "2450AT42A100" H 9950 5950 60  0000 C CNN
-F 2 "" H 9950 6050 60  0001 C CNN
+F 2 "hlib:2450AT42A100" H 9950 6050 60  0001 C CNN
 F 3 "" H 9950 6050 60  0000 C CNN
 F 4 "2450AT42A100" H 9950 6050 60  0001 C CNN "MPN"
@@
 F 0 "D1" H 2700 6450 50  0000 C CNN
 F 1 "BI_COLOR_LED" H 2700 6250 50  0000 C CNN
-F 2 "" H 2700 6350 60  0001 C CNN
+F 2 "hlib:APTB1612ESGC-F01" H 2700 6350 60  0001 C CNN
 F 3 "" H 2700 6350 60  0000 C CNN
 F 4 "APTB1612ESGC-F01" H 2700 6350 60  0001 C CNN "MPN"
@@
 F 0 "D1" H 2700 6800 50  0000 C CNN
 F 1 "BI_COLOR_LED" H 2700 6600 50  0000 C CNN
-F 2 "" H 2700 6700 60  0001 C CNN
+F 2 "hlib:APTB1612ESGC-F01" H 2700 6700 60  0001 C CNN
 F 3 "" H 2700 6700 60  0000 C CNN
 	2    2700 6700
