File: cad/smartercopter.sch (KiCad schematic (older format))
At the start: 29 parts, among them P1 CONN_5, P5 CONN_01X01, P6 CONN_01X01, P7 CONN_01X01, U1 CC2541, X1 32Mhz

Commit message: changed cc2451 footprint center pad
Parts:
- U1: footprint SMD_Packages:LFCSP-40-1EP -> hlib:VQFN-40
Changed lines of the file:
@@
 F 0 "U1" H 3650 4150 60  0000 C CNN
 F 1 "CC2541" H 3750 1000 60  0000 C CNN
-F 2 "SMD_Packages:LFCSP-40-1EP" H 4500 1250 60  0001 C CNN
+F 2 "hlib:VQFN-40" H 4500 1250 60  0001 C CNN
 F 3 "" H 4500 1250 60  0000 C CNN
 F 4 "CC2541F256RHAR" H 4100 2650 60  0001 C CNN "MPN"
