File: cad/smartercopter.kicad_pcb (KiCad board)
At the start: 2 copper layers, 37.7 x 16.8 mm, 74 parts, among them P1 CONN_5, P2 CONN_01X01, P3 CONN_01X01, P4 CONN_2, P5 CONN_01X01, P6 CONN_01X01, P7 CONN_01X01, Q1 SiA910EDJ, SW1 SW_PUSH_4, U1 CC2541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

Commit message: stuff on board
Parts:
- P1: moved to F.Cu
- moved D1 34.7 mm to (81.3, 115.4), turned to 180 degrees
- moved R2 30.1 mm to (79.0, 114.8), turned to 180 degrees
- moved R1 30.1 mm to (79.0, 116.1), turned to 180 degrees
- moved R3 11.7 mm to (72.3, 108.1)
- moved C9 11.0 mm to (70.4, 108.1), turned to 180 degrees
- moved R12 10.4 mm to (72.5, 109.2)
- moved R13 10.2 mm to (72.5, 110.2)
- moved P1 2.97 mm to (72.8, 105.8)
- moved SW1 2.01 mm to (81.9, 105.9)
- moved C12 0.59 mm to (55.5, 109.0)
- moved C13 0.59 mm to (55.5, 107.9)
- moved R7 0.59 mm to (54.0, 108.5)
- moved A1 0.50 mm to (56.3, 105.5)
- moved C20 0.36 mm to (64.2, 111.8)
- moved C22 0.36 mm to (66.4, 107.7)
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Routing:
- net Net-(D3-Pad2): track 7.69 -> 1.07 mm

Commit message: progress check in
Parts:
- moved C16 2.44 mm to (65.3, 119.6)
- moved C5 2.04 mm to (59.0, 114.9)
- moved C4 1.07 mm to (56.4, 114.0)
- moved C14 1.02 mm to (66.7, 115.5)
- moved C15 0.88 mm to (66.1, 112.7), turned to 180 degrees
- moved C3 0.58 mm to (53.5, 114.4)
- moved R4 0.47 mm to (60.3, 120.4)
- moved A1 0.45 mm to (56.3, 105.9)
- moved C2 0.43 mm to (57.8, 119.1)
- moved C22 0.27 mm to (66.4, 108.0)
- moved C1 0.17 mm to (53.1, 117.9)
- moved R5 0.16 mm to (61.3, 119.4)
- moved R1 0.15 mm to (78.9, 116.0)
- moved R2 0.13 mm to (78.9, 114.9)
- moved C9 0.09 mm to (70.5, 108.1)
Connections:
- C19 pad 1: Net-(C19-Pad1) -> /power/EN_REG
- D3 pad 3: Net-(C19-Pad1) -> /power/EN_REG
- R10 pad 1: Net-(C19-Pad1) -> /power/EN_REG
- U1 pad 32: /LED1 -> /LED2
- U1 pad 33: /LED2 -> /LED1
- U3 pad 3: /power/EN -> /power/EN_REG
- U4 pad 3: /power/EN -> /power/EN_REG
Routing:
- net /motor/EN: track 0.00 -> 29.3 mm, vias 0 -> 2
- net /motor/PH: track 0.00 -> 29.1 mm, vias 0 -> 2
- net /LED2: track 0.00 -> 28.2 mm, vias 0 -> 2
- net /LED1: track 0.00 -> 28.1 mm, vias 0 -> 2
- net /motor/UP_ROTOR: track 0.00 -> 28.0 mm
- net /motor/LOW_ROTOR: track 0.00 -> 26.5 mm, vias 0 -> 2
- net /motor/nSLEEP: track 0.00 -> 26.0 mm, vias 0 -> 2
- net /power/EN_REG: track 0.00 -> 25.9 mm, vias 0 -> 3
- net /power/EN: track 0.00 -> 21.9 mm, vias 0 -> 2
- net /power/BUTTON: track 2.55 -> 23.3 mm, vias 0 -> 2
- net Net-(C9-Pad1): track 0.00 -> 17.4 mm, vias 0 -> 2
- net /power/BATTVOLT: track 0.00 -> 15.6 mm
- net VCCA: track 6.07 -> 18.7 mm, vias 0 -> 6
- net Net-(D3-Pad2): track 1.07 -> 9.98 mm
- net +BATT: track 7.93 -> 13.3 mm
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
Commit message: more routing
Parts:
- moved C6 1.43 mm to (52.4, 110.8)
- moved C7 1.39 mm to (52.4, 109.9)
- moved R6 1.36 mm to (52.4, 112.1)
Routing:
- net /LED1: track 28.1 -> 0.95 mm, vias 2 -> 1
- net /LED2: track 28.2 -> 1.18 mm, vias 2 -> 1
- net /DD: track 0.00 -> 22.8 mm, vias 0 -> 1
- net /sensors/INT: track 0.00 -> 22.1 mm, vias 0 -> 2
- net /DC: track 0.00 -> 20.0 mm, vias 0 -> 1
- net VCCA: track 18.7 -> 21.6 mm
- net Net-(C9-Pad1): track 17.4 -> 15.8 mm
- net /motor/PH: track 29.1 -> 27.6 mm
- net /motor/LOW_ROTOR: track 26.5 -> 25.9 mm
